File: 379.kicad_pcb (KiCad board)
At the start: 2 copper layers, 342.6 x 92.7 mm, 176 parts, among them J1 DB, SW1 MX_SW_solder, SW10 MX_SW_solder, SW100 SW_Push, SW11 MX_SW_solder, SW12 MX_SW_solder, SW13 MX_SW_solder, SW14 MX_SW_solder, SW15 MX_SW_solder, SW16 MX_SW_solder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

Commit message: this bad boy is hot to go
Parts:
- moved J1 19.1 mm to (144.4, 37.0)
Routing:
- net D-: track 72.0 -> 92.2 mm
- net D+: track 71.3 -> 91.5 mm
- net +5V: track 11.3 -> 29.5 mm
- net GND: track 34.6 -> 18.1 mm
- net R1: track 342.8 -> 344.7 mm
Other:
- outline, holes or cut-outs redrawn
